Commit message: fixed format

File: mia_hand_description/materials/materials.xacro (robot description, xacro)
@@ -1,9 +1,9 @@
 <?xml version="1.0"?>
 <robot>
-    <material name="white">
-      <color rgba="1.0 1.0 1.0 1.0"/>
-    </material>
-    <material name="black">
-      <color rgba="0.0 0.0 0.0 1.0"/>
-    </material>
+  <material name="white">
+    <color rgba="1.0 1.0 1.0 1.0"/>
+  </material>
+  <material name="black">
+    <color rgba="0.0 0.0 0.0 1.0"/>
+  </material>
 </robot>
