Commit message: added mia hand

File: ur_simulation_gz/urdf/ur_gz.urdf.xacro (robot description, xacro)
@@ -2,11 +2,23 @@
 <robot xmlns:xacro="http://wiki.ros.org/xacro" name="$(arg name)">
   <!-- robot name parameter -->
-  <xacro:arg name="name" default="ur"/>
-  <!-- import main macro -->
+  <xacro:arg name="name" default="ur5e"/>
+  <!-- mia hand parameters -->
+  <xacro:arg name="serial_port" default="/dev/ttyUSB0"/>
+  <xacro:arg name="laterality" default="right" />
+  <!-- <xacro:arg name="joint_limits_config_file" default="$(find mia_hand_description)/calibration/joint_limits_default.yaml"/> -->
+  <xacro:arg name="joint_limits_config_file" default="joint_limits_default.yaml"/>
+  <xacro:arg name="prefix" default=""/>
+  <xacro:arg name="use_mock_hardware" default="true"/>
+  <!-- import ur5 macro -->
   <xacro:include filename="$(find ur_description)/urdf/ur_macro.xacro"/>
+  <!-- import ur5 ROS2 control macro -->
   <xacro:include filename="$(find ur_simulation_gz)/urdf/ur_gz.ros2_control.xacro" />
-  <!-- possible 'ur_type' values: ur3, ur3e, ur5, ur5e, ur7e, ur10, ur10e, ur12e, ur16e, ur8long, ur15, ur18, ur20, ur30 -->
+  <!-- import Mia Hand macro -->
+  <xacro:include filename="$(find mia_hand_description)/urdf/mia_hand.urdf.xacro"/>
+  <!-- import Mia Hand ROS2 control macro -->
+  <xacro:include filename="$(find mia_hand_description)/urdf/mia_hand.ros2_control.xacro"/>
+  <!-- possible 'ur_type' values: ur3, ur3e, ur5, ur5e, ur7e, ur10, ur10e, ur12e, ur16e, ur15, ur20, ur30 -->
   <!-- the default value should raise an error in case this was called without defining the type -->
-  <xacro:arg name="ur_type" default="ur5x"/>
+  <xacro:arg name="ur_type" default="ur5e"/>
   <!-- parameters -->
   <xacro:arg name="tf_prefix" default="" />
@@ -61,6 +73,19 @@
     <origin xyz="0 0 0" rpy="0 0 0" />          <!-- position robot in the world -->
   </xacro:ur_robot>
-  <gazebo reference="world">
-  </gazebo>
+  <!-- mia hand -->
+  <xacro:mia_hand
+    laterality="$(arg laterality)"
+    joint_limits_config_file="$(arg joint_limits_config_file)"
+    parent="tool0"
+    prefix="$(arg prefix)">
+    <xacro:if value="${'right' == '$(arg laterality)'}">
+      <origin xyz="0 0 0" rpy="1.59 0 0"/>
+    </xacro:if>
+    <xacro:if value="${'left' == '$(arg laterality)'}">
+      <origin xyz="0 0 0" rpy="1.57 3.14 0.1"/>
+    </xacro:if>
+  </xacro:mia_hand>
+  <!-- Gazebo specific elements -->
+  <gazebo reference="world"></gazebo>
   <gazebo>
     <plugin filename="gz_ros2_control-system" name="gz_ros2_control::GazeboSimROS2ControlPlugin">
@@ -77,3 +102,10 @@
     transmission_hw_interface="$(arg transmission_hw_interface)"
   />
+  <!-- mia hand ros2 control instance -->
+  <xacro:mia_hand_ros2_control
+    name="MiaHand"
+    prefix="$(arg prefix)"
+    serial_port="$(arg serial_port)"
+    use_mock_hardware="$(arg use_mock_hardware)"
+  />
 </robot>

Commit message: added cam

File: ur_simulation_gz/urdf/ur_gz.urdf.xacro (robot description, xacro)
@@ -18,4 +18,6 @@
   <!-- import Mia Hand ROS2 control macro -->
   <xacro:include filename="$(find mia_hand_description)/urdf/mia_hand.ros2_control.xacro"/>
+  <!-- import Camera macro -->
+  <xacro:include filename="$(find realsense2_description)/urdf/_d435.urdf.xacro"/>
   <!-- possible 'ur_type' values: ur3, ur3e, ur5, ur5e, ur7e, ur10, ur10e, ur12e, ur16e, ur15, ur20, ur30 -->
   <!-- the default value should raise an error in case this was called without defining the type -->
@@ -86,4 +88,11 @@
     </xacro:if>
   </xacro:mia_hand>
+   <!-- RealSense D435 Camera -->
+  <xacro:sensor_d435
+      name="camera"
+      parent="base_link">
+    <!-- relative Pose Kamera zu diesem Link -->
+    <origin xyz="0 0 1.30" rpy="0 0 0"/>
+  </xacro:sensor_d435>
   <!-- Gazebo specific elements -->
   <gazebo reference="world"></gazebo>

Commit message: added cam to rob model

File: ur_simulation_gz/urdf/ur_gz.urdf.xacro (robot description, xacro)
@@ -91,7 +91,10 @@
   <xacro:sensor_d435
       name="camera"
-      parent="base_link">
+      parent="base_link"
+      use_nominal_extrinsics="false"
+      add_plug="false"
+      use_mesh="true">
     <!-- relative Pose Kamera zu diesem Link -->
-    <origin xyz="0 0 1.30" rpy="0 0 0"/>
+    <origin xyz="0 0 1.30" rpy="0 1 1"/>
   </xacro:sensor_d435>
   <!-- Gazebo specific elements -->
@@ -105,4 +108,24 @@
     </plugin>
   </gazebo>
+  <!-- <gazebo reference="camera_depth_frame">
+    <sensor name="rgbd_camera" type="rgbd_camera">
+      <always_on>true</always_on>
+      <update_rate>5</update_rate>
+      <visualize>true</visualize>
+      <camera>
+        <horizontal_fov>1</horizontal_fov>
+        <image>
+          <width>640</width>
+          <height>480</height>
+          <format>R8G8B8</format>
+        </image>
+        <clip>
+          <near>0.05</near>
+          <far>3.0</far>
+        </clip>
+      </camera>
+      <topic>/rgbd_camera</topic>
+    </sensor>
+  </gazebo> -->
   <!-- ros2 control instance -->
   <xacro:ur_ros2_control

Commit message: added realsense mount rob model

File: ur_simulation_gz/urdf/ur_gz.urdf.xacro (robot description, xacro)
@@ -20,4 +20,6 @@
   <!-- import Camera macro -->
   <xacro:include filename="$(find realsense2_description)/urdf/_d435.urdf.xacro"/>
+  <!-- import Realsense Mount macro -->
+  <xacro:include filename="$(find ur_simulation_gz)/urdf/ur_realsense_mount.xacro"/>
   <!-- possible 'ur_type' values: ur3, ur3e, ur5, ur5e, ur7e, ur10, ur10e, ur12e, ur16e, ur15, ur20, ur30 -->
   <!-- the default value should raise an error in case this was called without defining the type -->
@@ -75,4 +77,9 @@
     <origin xyz="0 0 0" rpy="0 0 0" />          <!-- position robot in the world -->
   </xacro:ur_robot>
+  <xacro:ur_realsense_mount
+    parent_link="tool0"
+    xyz="0 0 0"
+    rpy="0 0 0">
+  </xacro:ur_realsense_mount>
   <!-- mia hand -->
   <xacro:mia_hand

File: ur_simulation_gz/urdf/ur_realsense_mount.xacro (robot description, xacro)
@@ -1,33 +1,33 @@
 <?xml version="1.0"?>
-<xacro:macro name="ur_realsense_mount" params="parent_link xyz rpy">
-  <!-- Neuer Link -->
-  <link name="custom_tool">
-    <visual>
+<robot xmlns:xacro="http://www.ros.org/wiki/xacro">
+  <xacro:macro name="ur_realsense_mount" params="parent_link xyz rpy">
+    <!-- Neuer Link -->
+    <link name="custom_tool">
+      <visual>
+        <origin xyz="${xyz}" rpy="${rpy}"/>
+        <geometry>
+          <mesh filename="$(find ur_simulation_gz)/meshes/halterung_realsense.stl" scale="0.001 0.001 0.001"/>
+        </geometry>
+      </visual>
+      <collision>
+        <origin xyz="${xyz}" rpy="${rpy}"/>
+        <geometry>
+          <mesh filename="$(find ur_simulation_gz)/meshes/halterung_realsense.stl" scale="0.001 0.001 0.001"/>
+        </geometry>
+      </collision>
+      <inertial>
+        <mass value="0.1"/>
+        <inertia
+          ixx="0.001" ixy="0" ixz="0"
+          iyy="0.001" iyz="0"
+          izz="0.001"/>
+      </inertial>
+    </link>
+    <!-- Fixed Joint -->
+    <joint name="custom_tool_joint" type="fixed">
+      <parent link="${parent_link}"/>
+      <child  link="custom_tool"/>
       <origin xyz="${xyz}" rpy="${rpy}"/>
-      <geometry>
-        <mesh filename="package://ur_simulation_gz/meshes/halterung_realsense.stl" scale="1 1 1"/>
-      </geometry>
-    </visual>
-    <collision>
-      <origin xyz="${xyz}" rpy="${rpy}"/>
-      <geometry>
-        <mesh filename="package://ur_simulation_gz/meshes/halterung_realsense.stl" scale="1 1 1"/>
-      </geometry>
-    </collision>
-    <inertial>
-      <mass value="0.1"/>
-      <origin xyz="0 0 0" rpy="0 0 0"/>
-      <inertia
-        ixx="0.001" ixy="0" ixz="0"
-        iyy="0.001" iyz="0"
-        izz="0.001"/>
-      </inertia>
-    </inertial>
-  </link>
-  <!-- Fixed Joint -->
-  <joint name="custom_tool_joint" type="fixed">
-    <parent link="${parent_link}"/>
-    <child  link="custom_tool"/>
-    <origin xyz="${xyz}" rpy="${rpy}"/>
-  </joint>
-</xacro:macro>
+    </joint>
+  </xacro:macro>
+</robot>
