Commit message: changed folder names

File: manipulator_moveit_config/srdf/manipulator.srdf.xacro (robot description, xacro)
@@ -3,5 +3,5 @@
   <!-- robot name parameter -->
   <xacro:arg name="name" default="ur5e"/>
-  <xacro:include filename="$(find ur5_mia_moveit_config)/srdf/ur_macro.srdf.xacro"/>
-  <xacro:ur_srdf/>
+  <xacro:include filename="$(find ur5_mia_moveit_config)/srdf/manipulator_macro.srdf.xacro"/>
+  <xacro:manipulator_srdf/>
 </robot>

File: manipulator_moveit_config/srdf/manipulator_macro.srdf.xacro (robot description, xacro)
@@ -5,5 +5,5 @@
     A URDF file must exist for this robot as well, where the joints and the links that are referenced are defined
 -->
-  <xacro:macro name="ur_srdf" params="">
+  <xacro:macro name="manipulator_srdf" params="">
     <!--GROUPS - Representation of a set of joints and links. This can be useful for specifying DOF to plan for, defining arms, end effectors, etc-->
     <!--LINKS - When a link is specified, the parent joint of that link (if it exists) is automatically included-->
