Commit message: changed color camera mount

File: manipulator_description/urdf/ur_realsense_mount.xacro (robot description, xacro)
@@ -9,4 +9,5 @@
           <mesh filename="package://manipulator_description/meshes/halterung_realsense.stl" scale="0.001 0.001 0.001"/>
         </geometry>
+        <material name="MYBLACK"/>
       </visual>
       <collision>
@@ -30,4 +31,7 @@
       <origin xyz="${xyz}" rpy="${rpy}"/>
     </joint>
+    <material name="MYBLACK">
+		  <color rgba="0.01568627450980392 0.01568627450980392 0.01568627450980392 1.0"/>
+	  </material>
   </xacro:macro>
 </robot>
