Commit message: fixed simulation launch

File: manipulator_description/urdf/manipulator_gz.urdf.xacro (robot description, xacro)
@@ -131,5 +131,5 @@
   <!-- ros2 control instance -->
   <xacro:ur_ros2_control
-    name="$(arg name)"
+    name="$(arg ur_type)"
     tf_prefix="$(arg tf_prefix)"
     transmission_hw_interface="$(arg transmission_hw_interface)"

File: manipulator_description/urdf/ur_realsense_mount.xacro (robot description, xacro)
@@ -7,5 +7,5 @@
         <origin xyz="${xyz}" rpy="${rpy}"/>
         <geometry>
-          <mesh filename="$(find ur_simulation_gz)/meshes/halterung_realsense.stl" scale="0.001 0.001 0.001"/>
+          <mesh filename="package://manipulator_description/meshes/halterung_realsense.stl" scale="0.001 0.001 0.001"/>
         </geometry>
       </visual>
@@ -13,5 +13,5 @@
         <origin xyz="${xyz}" rpy="${rpy}"/>
         <geometry>
-          <mesh filename="$(find ur_simulation_gz)/meshes/halterung_realsense.stl" scale="0.001 0.001 0.001"/>
+          <mesh filename="package://manipulator_description/meshes/halterung_realsense.stl" scale="0.001 0.001 0.001"/>
         </geometry>
       </collision>

File: manipulator_moveit_config/srdf/manipulator.srdf.xacro (robot description, xacro)
@@ -3,5 +3,5 @@
   <!-- robot name parameter -->
   <xacro:arg name="name" default="ur5e"/>
-  <xacro:include filename="$(find ur5_mia_moveit_config)/srdf/manipulator_macro.srdf.xacro"/>
+  <xacro:include filename="$(find manipulator_moveit_config)/srdf/manipulator_macro.srdf.xacro"/>
   <xacro:manipulator_srdf/>
 </robot>

Commit message: fixed errors sim

File: manipulator_description/urdf/manipulator_gz.urdf.xacro (robot description, xacro)
@@ -81,5 +81,5 @@
     laterality="$(arg laterality)"
     joint_limits_config_file="$(arg joint_limits_config_file)"
-    parent="tool0"
+    parent="ur_realsense_mount_link"
     prefix="$(arg prefix)">
     <xacro:if value="${'right' == '$(arg laterality)'}">

File: manipulator_description/urdf/ur_realsense_mount.xacro (robot description, xacro)
@@ -3,5 +3,5 @@
   <xacro:macro name="ur_realsense_mount" params="parent_link xyz rpy">
     <!-- Neuer Link -->
-    <link name="custom_tool">
+    <link name="ur_realsense_mount_link">
       <visual>
         <origin xyz="${xyz}" rpy="${rpy}"/>
@@ -25,7 +25,7 @@
     </link>
     <!-- Fixed Joint -->
-    <joint name="custom_tool_joint" type="fixed">
+    <joint name="ur_realsense_mount_joint" type="fixed">
       <parent link="${parent_link}"/>
-      <child  link="custom_tool"/>
+      <child  link="ur_realsense_mount_link"/>
       <origin xyz="${xyz}" rpy="${rpy}"/>
     </joint>

File: manipulator_moveit_config/srdf/manipulator_macro.srdf.xacro (robot description, xacro)
@@ -82,4 +82,8 @@
     <disable_collisions link1="middle_fle" link2="palm" reason="Adjacent"/>
     <disable_collisions link1="ring_fle" link2="palm" reason="Adjacent"/>
+    <disable_collisions link1="ur_realsense_mount_link" link2="tool0" reason="Adjacent"/>
+    <disable_collisions link1="ur_realsense_mount_link" link2="wrist_3_link" reason="Adjacent"/>
+    <disable_collisions link1="ur_realsense_mount_link" link2="palm" reason="Adjacent"/>
+    <disable_collisions link1="ur_realsense_mount_link" link2="hand_ee_link" reason="Adjacent"/>
   </xacro:macro>
 </robot>

Commit message: added schrank in scene

File: manipulator_description/urdf/manipulator_gz.urdf.xacro (robot description, xacro)
@@ -13,4 +13,6 @@
   <!-- import Realsense Mount macro -->
   <xacro:include filename="$(find manipulator_description)/urdf/ur_realsense_mount.xacro"/>
+  <!-- import Scene Objects macro -->
+  <xacro:include filename="$(find manipulator_description)/urdf/schrankregal.xacro"/>
   <!-- possible 'ur_type' values: ur3, ur3e, ur5, ur5e, ur7e, ur10, ur10e, ur12e, ur16e, ur15, ur20, ur30 -->
   <!-- the default value should raise an error in case this was called without defining the type -->
@@ -57,4 +59,10 @@
     <child link="ground_plane"/>
   </joint>
+  <!-- scene -->
+  <xacro:schrankregal
+    parent_link="world"
+    xyz="-0.42 0.42 0"
+    rpy="1.571 0 -0.960">
+  </xacro:schrankregal>
   <!-- arm -->
   <xacro:ur_robot
@@ -84,5 +92,5 @@
     prefix="$(arg prefix)">
     <xacro:if value="${'right' == '$(arg laterality)'}">
-      <origin xyz="0 0 0" rpy="1.59 0 0"/>
+      <origin xyz="0 0 0" rpy="1.59 0 1.59"/>
     </xacro:if>
     <xacro:if value="${'left' == '$(arg laterality)'}">
@@ -98,4 +106,13 @@
       use_mesh="true">
     <origin xyz="0 0 1.30" rpy="0 1 1"/>
+  </xacro:sensor_d435>
+  <!-- RealSense D435 Camera Tool-->
+  <xacro:sensor_d435
+      name="camera_tool"
+      parent="tool0"
+      use_nominal_extrinsics="false"
+      add_plug="false"
+      use_mesh="true">
+    <origin xyz="0 0.135 0.012" rpy="0 -1.57 1.57"/>
   </xacro:sensor_d435>
   <!-- Gazebo specific elements -->

File: manipulator_moveit_config/srdf/manipulator_macro.srdf.xacro (robot description, xacro)
@@ -86,4 +86,5 @@
     <disable_collisions link1="ur_realsense_mount_link" link2="palm" reason="Adjacent"/>
     <disable_collisions link1="ur_realsense_mount_link" link2="hand_ee_link" reason="Adjacent"/>
+    <disable_collisions link1="ur_realsense_mount_link" link2="camera_tool_link" reason="Adjacent"/>
   </xacro:macro>
 </robot>

Commit message: edit sensor3d

File: manipulator_description/urdf/manipulator_gz.urdf.xacro (robot description, xacro)
@@ -114,15 +114,15 @@
   </xacro:mia_hand>
    <!-- RealSense D435 Camera -->
-  <!-- <xacro:sensor_d435
-      name="camera_base"
+  <xacro:sensor_d435
+      name="camera"
       parent="base_link"
       use_nominal_extrinsics="false"
       add_plug="false"
       use_mesh="true">
-    <origin xyz="0 0 1.30" rpy="0 1 1"/>
-  </xacro:sensor_d435> -->
+    <origin xyz="0.35 -0.35 0.57" rpy="0 0 2.35619"/>
+  </xacro:sensor_d435>
   <!-- RealSense D435 Camera Tool-->
-  <xacro:sensor_d435
-      name="camera_tool"
+  <!-- <xacro:sensor_d435
+      name="camera"
       parent="tool0"
       use_nominal_extrinsics="false"
@@ -130,5 +130,5 @@
       use_mesh="true">
     <origin xyz="0 0.135 0.012" rpy="0 -1.57 1.57"/>
-  </xacro:sensor_d435>
+  </xacro:sensor_d435> -->
   <!-- Gazebo specific elements -->
   <gazebo reference="world"></gazebo>
