Commit message: changed naming

File: manipulator_description/urdf/manipulator.urdf.xacro (robot description, xacro)
@@ -12,5 +12,5 @@
   <xacro:include filename="$(find realsense2_description)/urdf/_d435.urdf.xacro"/>
   <!-- import Realsense Mount macro -->
-  <xacro:include filename="$(find ur_simulation_gz)/urdf/ur_realsense_mount.xacro"/>
+  <xacro:include filename="$(find manipulator_description)/urdf/ur_realsense_mount.xacro"/>
   <!-- ur5 parameters -->
   <!-- possible 'ur_type' values: ur3, ur3e, ur5, ur5e, ur7e, ur10, ur10e, ur12e, ur16e, ur15, ur20, ur30 -->
@@ -18,5 +18,5 @@
   <xacro:arg name="ur_type" default="ur5e"/>
   <xacro:arg name="tf_prefix" default="" />
-  <xacro:arg name="joint_limit_params" default="$(find ur_simulation_gz)/config/ur_joint_limits.yaml"/>
+  <xacro:arg name="joint_limit_params" default="$(find manipulator_description)/config/ur_joint_limits.yaml"/>
   <xacro:arg name="kinematics_params" default="$(find ur_description)/config/$(arg ur_type)/default_kinematics.yaml"/>
   <xacro:arg name="physical_params" default="$(find ur_description)/config/$(arg ur_type)/physical_parameters.yaml"/>
@@ -74,7 +74,6 @@
     safety_pos_margin="$(arg safety_pos_margin)"
     safety_k_position="$(arg safety_k_position)"
-    force_abs_paths="true"
-    >
-    <origin xyz="0 0 0" rpy="0 0 0" />          <!-- position robot in the world -->
+    force_abs_paths="true">
+    <origin xyz="0 0 0" rpy="0 0 0" />
   </xacro:ur_robot>
   <xacro:ur_realsense_mount
@@ -103,5 +102,4 @@
       add_plug="false"
       use_mesh="true">
-    <!-- relative Pose Kamera zu diesem Link -->
     <origin xyz="0 0 1.30" rpy="0 1 1"/>
   </xacro:sensor_d435>

File: manipulator_description/urdf/manipulator_gz.urdf.xacro (robot description, xacro)
@@ -4,5 +4,5 @@
   <xacro:include filename="$(find ur_description)/urdf/ur_macro.xacro"/>
   <!-- import ur5 ROS2 control macro -->
-  <xacro:include filename="$(find ur_robot_driver)/urdf/ur.ros2_control.xacro"/>
+  <xacro:include filename="$(find ur_simulation_gz)/urdf/ur_gz.ros2_control.xacro" />
   <!-- import Mia Hand macro -->
   <xacro:include filename="$(find mia_hand_description)/urdf/mia_hand.urdf.xacro"/>
@@ -12,24 +12,19 @@
   <xacro:include filename="$(find realsense2_description)/urdf/_d435.urdf.xacro"/>
   <!-- import Realsense Mount macro -->
-  <xacro:include filename="$(find ur_simulation_gz)/urdf/ur_realsense_mount.xacro"/>
-  <!-- ur5 parameters -->
+  <xacro:include filename="$(find manipulator_description)/urdf/ur_realsense_mount.xacro"/>
   <!-- possible 'ur_type' values: ur3, ur3e, ur5, ur5e, ur7e, ur10, ur10e, ur12e, ur16e, ur15, ur20, ur30 -->
   <!-- the default value should raise an error in case this was called without defining the type -->
   <xacro:arg name="ur_type" default="ur5e"/>
   <xacro:arg name="tf_prefix" default="" />
-  <xacro:arg name="joint_limit_params" default="$(find ur_simulation_gz)/config/ur_joint_limits.yaml"/>
+  <xacro:arg name="joint_limit_params" default="$(find manipulator_description)/config/ur_joint_limits.yaml"/>
   <xacro:arg name="kinematics_params" default="$(find ur_description)/config/$(arg ur_type)/default_kinematics.yaml"/>
   <xacro:arg name="physical_params" default="$(find ur_description)/config/$(arg ur_type)/physical_parameters.yaml"/>
   <xacro:arg name="visual_params" default="$(find ur_description)/config/$(arg ur_type)/visual_parameters.yaml"/>
-  <xacro:arg name="robot_ip" default="0.0.0.0"/>
-  <xacro:arg name="headless_mode" default="false" />
-  <xacro:arg name="ur_script_filename" default="$(find ur_client_library)/resources/external_control.urscript"/>
-  <xacro:arg name="ur_output_recipe_filename" default="$(find ur_robot_driver)/resources/rtde_output_recipe.txt"/>
-  <xacro:arg name="ur_input_recipe_filename" default="$(find ur_robot_driver)/resources/rtde_input_recipe.txt"/>
+  <xacro:arg name="transmission_hw_interface" default=""/>
   <xacro:arg name="safety_limits" default="false"/>
   <xacro:arg name="safety_pos_margin" default="0.15"/>
   <xacro:arg name="safety_k_position" default="20"/>
-  <xacro:arg name="use_mock_hardware" default="false" />
-  <xacro:arg name="mock_sensor_commands" default="false" />
+  <xacro:arg name="simulation_controllers" default="" />
+  <xacro:arg name="ros_namespace" default="" />
   <!-- mia hand parameters -->
   <xacro:arg name="serial_port" default="/dev/ttyUSB0"/>
@@ -37,5 +32,5 @@
   <xacro:arg name="joint_limits_config_file" default="joint_limits_default.yaml"/>
   <xacro:arg name="prefix" default=""/>
-  <xacro:arg name="mia_use_mock_hardware" default="true"/>
+  <xacro:arg name="use_mock_hardware" default="true"/>
   <!-- create link fixed to the "world" -->
   <link name="world" />
@@ -74,7 +69,6 @@
     safety_pos_margin="$(arg safety_pos_margin)"
     safety_k_position="$(arg safety_k_position)"
-    force_abs_paths="true"
-    >
-    <origin xyz="0 0 0" rpy="0 0 0" />          <!-- position robot in the world -->
+    force_abs_paths="true">
+    <origin xyz="0 0 0" rpy="0 0 0" />
   </xacro:ur_robot>
   <xacro:ur_realsense_mount
@@ -103,19 +97,41 @@
       add_plug="false"
       use_mesh="true">
-    <!-- relative Pose Kamera zu diesem Link -->
     <origin xyz="0 0 1.30" rpy="0 1 1"/>
   </xacro:sensor_d435>
+  <!-- Gazebo specific elements -->
+  <gazebo reference="world"></gazebo>
+  <gazebo>
+    <plugin filename="gz_ros2_control-system" name="gz_ros2_control::GazeboSimROS2ControlPlugin">
+      <parameters>$(arg simulation_controllers)</parameters>
+      <ros>
+        <namespace>$(arg ros_namespace)</namespace>
+      </ros>
+    </plugin>
+  </gazebo>
+  <!-- <gazebo reference="camera_depth_frame">
+    <sensor name="rgbd_camera" type="rgbd_camera">
+      <always_on>true</always_on>
+      <update_rate>5</update_rate>
+      <visualize>true</visualize>
+      <camera>
+        <horizontal_fov>1</horizontal_fov>
+        <image>
+          <width>640</width>
+          <height>480</height>
+          <format>R8G8B8</format>
+        </image>
+        <clip>
+          <near>0.05</near>
+          <far>3.0</far>
+        </clip>
+      </camera>
+      <topic>/rgbd_camera</topic>
+    </sensor>
+  </gazebo> -->
   <!-- ros2 control instance -->
   <xacro:ur_ros2_control
-    name="$(arg ur_type)"
+    name="$(arg name)"
     tf_prefix="$(arg tf_prefix)"
-    kinematics_parameters_file="$(arg kinematics_params)"
-    robot_ip="$(arg robot_ip)"
-    script_filename="$(arg ur_script_filename)"
-    output_recipe_filename="$(arg ur_output_recipe_filename)"
-    input_recipe_filename="$(arg ur_input_recipe_filename)"
-    use_mock_hardware="$(arg use_mock_hardware)"
-    mock_sensor_commands="$(arg mock_sensor_commands)"
-    headless_mode="$(arg headless_mode)"
+    transmission_hw_interface="$(arg transmission_hw_interface)"
   />
   <!-- mia hand ros2 control instance -->
@@ -124,5 +140,5 @@
     prefix="$(arg prefix)"
     serial_port="$(arg serial_port)"
-    use_mock_hardware="$(arg mia_use_mock_hardware)"
+    use_mock_hardware="$(arg use_mock_hardware)"
   />
 </robot>

Commit message: changed mia hand rot

File: manipulator_description/urdf/manipulator.urdf.xacro (robot description, xacro)
@@ -13,4 +13,6 @@
   <!-- import Realsense Mount macro -->
   <xacro:include filename="$(find manipulator_description)/urdf/ur_realsense_mount.xacro"/>
+  <!-- import Scene Objects macro -->
+  <xacro:include filename="$(find manipulator_description)/urdf/schrankregal.xacro"/>
   <!-- ur5 parameters -->
   <!-- possible 'ur_type' values: ur3, ur3e, ur5, ur5e, ur7e, ur10, ur10e, ur12e, ur16e, ur15, ur20, ur30 -->
@@ -62,4 +64,10 @@
     <child link="ground_plane"/>
   </joint>
+    <!-- scene -->
+  <xacro:schrankregal
+    parent_link="world"
+    xyz="-0.42 0.42 0"
+    rpy="1.571 0 -0.960">
+  </xacro:schrankregal>
   <!-- arm -->
   <xacro:ur_robot
@@ -89,5 +97,5 @@
     prefix="$(arg prefix)">
     <xacro:if value="${'right' == '$(arg laterality)'}">
-      <origin xyz="0 0 0" rpy="1.59 0 0"/>
+      <origin xyz="0 0 0" rpy="1.59 0 1.59"/>
     </xacro:if>
     <xacro:if value="${'left' == '$(arg laterality)'}">
@@ -103,4 +111,13 @@
       use_mesh="true">
     <origin xyz="0 0 1.30" rpy="0 1 1"/>
+  </xacro:sensor_d435>
+    <!-- RealSense D435 Camera Tool-->
+  <xacro:sensor_d435
+      name="camera_tool"
+      parent="tool0"
+      use_nominal_extrinsics="false"
+      add_plug="false"
+      use_mesh="true">
+    <origin xyz="0 0.135 0.012" rpy="0 -1.57 1.57"/>
   </xacro:sensor_d435>
   <!-- ros2 control instance -->

File: manipulator_description/urdf/manipulator_gz.urdf.xacro (robot description, xacro)
@@ -99,6 +99,6 @@
   </xacro:mia_hand>
    <!-- RealSense D435 Camera -->
-  <xacro:sensor_d435
-      name="camera"
+  <!-- <xacro:sensor_d435
+      name="camera_base"
       parent="base_link"
       use_nominal_extrinsics="false"
@@ -106,8 +106,8 @@
       use_mesh="true">
     <origin xyz="0 0 1.30" rpy="0 1 1"/>
-  </xacro:sensor_d435>
+  </xacro:sensor_d435> -->
   <!-- RealSense D435 Camera Tool-->
   <xacro:sensor_d435
-      name="camera_tool"
+      name="camera"
       parent="tool0"
       use_nominal_extrinsics="false"

Commit message: added regal

File: manipulator_description/urdf/manipulator.urdf.xacro (robot description, xacro)
@@ -64,8 +64,23 @@
     <child link="ground_plane"/>
   </joint>
-    <!-- scene -->
+  <!-- scene -->
   <xacro:schrankregal
+    name="unten"
     parent_link="world"
     xyz="-0.42 0.42 0"
+    rpy="1.571 0 -0.960">
+  </xacro:schrankregal>
+  <!-- scene -->
+  <xacro:schrankregal
+    name="mitte"
+    parent_link="world"
+    xyz="-0.42 0.42 0.46"
+    rpy="1.571 0 -0.960">
+  </xacro:schrankregal>
+  <!-- scene -->
+  <xacro:schrankregal
+    name="oben"
+    parent_link="world"
+    xyz="-0.42 0.42 0.92"
     rpy="1.571 0 -0.960">
   </xacro:schrankregal>

File: manipulator_description/urdf/manipulator_gz.urdf.xacro (robot description, xacro)
@@ -61,6 +61,21 @@
   <!-- scene -->
   <xacro:schrankregal
+    name="unten"
     parent_link="world"
     xyz="-0.42 0.42 0"
+    rpy="1.571 0 -0.960">
+  </xacro:schrankregal>
+  <!-- scene -->
+  <xacro:schrankregal
+    name="mitte"
+    parent_link="world"
+    xyz="-0.42 0.42 0.46"
+    rpy="1.571 0 -0.960">
+  </xacro:schrankregal>
+  <!-- scene -->
+  <xacro:schrankregal
+    name="oben"
+    parent_link="world"
+    xyz="-0.42 0.42 0.92"
     rpy="1.571 0 -0.960">
   </xacro:schrankregal>

File: manipulator_description/urdf/schrankregal.xacro (robot description, xacro)
@@ -1,7 +1,7 @@
 <?xml version="1.0"?>
 <robot xmlns:xacro="http://www.ros.org/wiki/xacro">
-  <xacro:macro name="schrankregal" params="parent_link xyz rpy">
+  <xacro:macro name="schrankregal" params="name parent_link xyz rpy">
     <!-- Neuer Link -->
-    <link name="schrankregal_link">
+    <link name="${name}_schrankregal_link">
       <visual>
         <origin xyz="${xyz}" rpy="${rpy}"/>
@@ -9,5 +9,5 @@
           <mesh filename="package://manipulator_description/meshes/SchrankRegal.stl" scale="0.001 0.001 0.001"/>
         </geometry>
-        <material name="REGALCOLOR"/>
+        <material name="${name}_REGALCOLOR"/>
       </visual>
       <collision>
@@ -19,10 +19,10 @@
     </link>
     <!-- Fixed Joint -->
-    <joint name="schrankregal_joint" type="fixed">
+    <joint name="${name}_schrankregal_joint" type="fixed">
       <parent link="${parent_link}"/>
-      <child  link="schrankregal_link"/>
+      <child  link="${name}_schrankregal_link"/>
       <origin xyz="0 0 0" rpy="0 0 0"/>
     </joint>
-    <material name="REGALCOLOR">
+    <material name="${name}_REGALCOLOR">
 		  <color rgba="1 0.1686 0.6 1"/>
 	  </material>

File: manipulator_moveit_config/srdf/manipulator_macro.srdf.xacro (robot description, xacro)
@@ -86,5 +86,5 @@
     <disable_collisions link1="ur_realsense_mount_link" link2="palm" reason="Adjacent"/>
     <disable_collisions link1="ur_realsense_mount_link" link2="hand_ee_link" reason="Adjacent"/>
-    <disable_collisions link1="ur_realsense_mount_link" link2="camera_tool_link" reason="Adjacent"/>
+    <disable_collisions link1="ur_realsense_mount_link" link2="camera_link" reason="Adjacent"/>
   </xacro:macro>
 </robot>

Commit message: camera position adjusted

File: manipulator_description/urdf/manipulator.urdf.xacro (robot description, xacro)
@@ -156,5 +156,5 @@
       add_plug="false"
       use_mesh="true">
-    <origin xyz="0 0.135 0.012" rpy="0 -1.57 1.57"/>
+    <origin xyz="0 0.110 0.012" rpy="0 -1.57 -1.57"/>
   </xacro:sensor_d435>
   <!-- ros2 control instance -->
